File: ecad/BreadBoard-POC/BreadBoard-PoC.kicad_pcb (KiCad board)
At the start: 2 copper layers, 160 x 100 mm, 100 parts, among them J1 Conn_01x01, J10 Conn_01x01, J11 Conn_01x01, J12 Conn_01x01, J13 Conn_01x01, J14 Conn_01x01, J15 Conn_01x01, J16 Conn_01x01, J2 Conn_01x01, J3 Conn_01x01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

Commit message: Finalizing POC placement and routing.
Parts:
- added C45: 100n, Capacitor_THT:C_Rect_L4.6mm_W2.0mm_P2.50mm_MKS02_FKP02, F.Cu at (43.2, 91.4)
- added C46: 100n, Capacitor_THT:C_Rect_L4.6mm_W2.0mm_P2.50mm_MKS02_FKP02, F.Cu at (78.7, 91.4)
- added C47: 100n, Capacitor_THT:C_Rect_L4.6mm_W2.0mm_P2.50mm_MKS02_FKP02, F.Cu at (114.3, 91.4)
- added C48: 100n, Capacitor_THT:C_Rect_L4.6mm_W2.0mm_P2.50mm_MKS02_FKP02, F.Cu at (149.9, 91.4)
- added C49: 100n, Capacitor_THT:C_Rect_L4.6mm_W2.0mm_P2.50mm_MKS02_FKP02, F.Cu at (111.7, 111.8)
- added C50: 100n, Capacitor_THT:C_Rect_L4.6mm_W2.0mm_P2.50mm_MKS02_FKP02, F.Cu at (109.3, 124.5)
- added C52: 100n, Capacitor_THT:C_Rect_L4.6mm_W2.0mm_P2.50mm_MKS02_FKP02, F.Cu at (129.6, 114.3)
- added C53: 100u, Capacitor_THT:CP_Radial_D6.3mm_P2.50mm, F.Cu at (144.8, 116.9)
- added C54: 100n, Capacitor_THT:C_Rect_L4.6mm_W2.0mm_P2.50mm_MKS02_FKP02, F.Cu at (121.9, 129.5)
- added C55: 100n, Capacitor_THT:C_Rect_L4.6mm_W2.0mm_P2.50mm_MKS02_FKP02, F.Cu at (119.4, 129.5)
- added C56: 100n, Capacitor_THT:C_Rect_L4.6mm_W2.0mm_P2.50mm_MKS02_FKP02, F.Cu at (116.8, 129.5)
- added C57: 100n, Capacitor_THT:C_Rect_L4.6mm_W2.0mm_P2.50mm_MKS02_FKP02, F.Cu at (134.6, 129.5)
- added C58: 100n, Capacitor_THT:C_Rect_L4.6mm_W2.0mm_P2.50mm_MKS02_FKP02, F.Cu at (132.1, 129.5)
- added C59: 100n, Capacitor_THT:C_Rect_L4.6mm_W2.0mm_P2.50mm_MKS02_FKP02, F.Cu at (129.5, 129.5)
- added J17: AVR-ISP-6, Connector_PinHeader_2.54mm:PinHeader_2x03_P2.54mm_Vertical, F.Cu at (106.7, 129.5)
- added J18: Conn_01x04, Connector_PinHeader_2.54mm:PinHeader_1x04_P2.54mm_Vertical, F.Cu at (137.2, 114.3)
- added J19: Conn_01x04, Connector_PinHeader_2.54mm:PinHeader_1x04_P2.54mm_Vertical, F.Cu at (114.3, 137.2)
- added J20: Conn_01x04, Connector_PinHeader_2.54mm:PinHeader_1x04_P2.54mm_Vertical, F.Cu at (127.0, 137.2)
- added J21: Conn_01x01, Connector_PinHeader_2.54mm:PinHeader_1x01_P2.54mm_Vertical, F.Cu at (185.4, 63.5)
- added J22: Conn_01x01, Connector_PinHeader_2.54mm:PinHeader_1x01_P2.54mm_Vertical, F.Cu at (185.4, 86.4)
- added R25: 4K7, Resistor_THT:R_Axial_DIN0207_L6.3mm_D2.5mm_P2.54mm_Vertical, F.Cu at (78.8, 119.4)
- added R26: 10K, Resistor_THT:R_Axial_DIN0207_L6.3mm_D2.5mm_P2.54mm_Vertical, F.Cu at (43.2, 94.0)
- added R27: 10K, Resistor_THT:R_Axial_DIN0207_L6.3mm_D2.5mm_P2.54mm_Vertical, F.Cu at (78.7, 94.0)
- added R28: 10K, Resistor_THT:R_Axial_DIN0207_L6.3mm_D2.5mm_P2.54mm_Vertical, F.Cu at (114.3, 94.0)
- added R29: 10K, Resistor_THT:R_Axial_DIN0207_L6.3mm_D2.5mm_P2.54mm_Vertical, F.Cu at (149.9, 94.0)
- added R30: 33R, Resistor_THT:R_Axial_DIN0207_L6.3mm_D2.5mm_P2.54mm_Vertical, F.Cu at (101.6, 129.5)
- added R31: 33R, Resistor_THT:R_Axial_DIN0207_L6.3mm_D2.5mm_P2.54mm_Vertical, F.Cu at (99.1, 134.6)
- added R32: 10k, Resistor_THT:R_Axial_DIN0207_L6.3mm_D2.5mm_P2.54mm_Vertical, F.Cu at (132.1, 111.8)
- added R36: 4K7, Resistor_THT:R_Axial_DIN0207_L6.3mm_D2.5mm_P2.54mm_Vertical, F.Cu at (121.9, 134.6)
- added R37: 4K7, Resistor_THT:R_Axial_DIN0207_L6.3mm_D2.5mm_P2.54mm_Vertical, F.Cu at (119.4, 134.6)
- added R38: 4K7, Resistor_THT:R_Axial_DIN0207_L6.3mm_D2.5mm_P2.54mm_Vertical, F.Cu at (116.8, 134.6)
- added R42: 4K7, Resistor_THT:R_Axial_DIN0207_L6.3mm_D2.5mm_P2.54mm_Vertical, F.Cu at (129.5, 134.6)
- added R43: 4K7, Resistor_THT:R_Axial_DIN0207_L6.3mm_D2.5mm_P2.54mm_Vertical, F.Cu at (132.1, 134.6)
- added R44: 4K7, Resistor_THT:R_Axial_DIN0207_L6.3mm_D2.5mm_P2.54mm_Vertical, F.Cu at (134.6, 134.6)
- added RN1: R_Network08, Resistor_THT:R_Array_SIP9, F.Cu at (114.3, 142.2)
- added RV1: 1K, Potentiometer_THT:Potentiometer_Bourns_3266W_Vertical, F.Cu at (73.7, 119.4)
- added U5: ATmega328-P, Package_DIP:DIP-28_W7.62mm_LongPads, F.Cu at (127.0, 114.3)
- R11, R12, R17, R18, R23, R24, R5, R6: value 0R1 -> 0R5
Connections:
- C21 pad 1: /Driver_X2/VREF -> /Driver_X1/VREF
- C22 pad 1: /Driver_X2/VREF -> /Driver_X1/VREF
- C32 pad 1: /Driver_Y/VREF -> /Driver_X1/VREF
- C33 pad 1: /Driver_Y/VREF -> /Driver_X1/VREF
- C43 pad 1: /Driver_Z/VREF -> /Driver_X1/VREF
- C44 pad 1: /Driver_Z/VREF -> /Driver_X1/VREF
- R14 pad 1: /Driver_Y/EN -> /EN
- R2 pad 1: /Driver_X1/EN -> /EN
- R20 pad 1: /Driver_Z/EN -> /EN
- R8 pad 1: /Driver_X2/EN -> /EN
- U1 pad 1: /Driver_X1/STEP -> /STEP_X
- U1 pad 2: /Driver_X1/DIR -> /DIR_X
- U1 pad 23: /Driver_X1/RESET -> Net-(U1-RESET)
- U2 pad 1: /Driver_X2/STEP -> /STEP_X
- U2 pad 11: /Driver_X2/VREF -> /Driver_X1/VREF
- U2 pad 2: /Driver_X2/DIR -> /DIR_X
- U2 pad 23: /Driver_X2/RESET -> Net-(U2-RESET)
- U2 pad 24: /Driver_X2/VREF -> /Driver_X1/VREF
- U3 pad 1: /Driver_Y/STEP -> /STEP_Y
- U3 pad 11: /Driver_Y/VREF -> /Driver_X1/VREF
- U3 pad 2: /Driver_Y/DIR -> /DIR_Y
- U3 pad 23: /Driver_Y/RESET -> Net-(U3-RESET)
- U3 pad 24: /Driver_Y/VREF -> /Driver_X1/VREF
- U4 pad 1: /Driver_Z/STEP -> /STEP_Z
- U4 pad 11: /Driver_Z/VREF -> /Driver_X1/VREF
- U4 pad 2: /Driver_Z/DIR -> /DIR_Z
- U4 pad 23: /Driver_Z/RESET -> Net-(U4-RESET)
- U4 pad 24: /Driver_Z/VREF -> /Driver_X1/VREF
Routing:
- net +5V: track 0.00 -> 282.0 mm, vias 0 -> 2
- net GND: track 874.1 -> 1049.4 mm, vias 16 -> 28
- net /Driver_X1/VREF: track 10.2 -> 71.5 mm, vias 0 -> 16
- net Net-(U4-RESET): track 0.00 -> 22.9 mm, vias 0 -> 2
- net Net-(U1-RESET): track 0.00 -> 22.9 mm, vias 0 -> 2
- net Net-(U2-RESET): track 0.00 -> 22.9 mm, vias 0 -> 2
- net /SPI_MOSI: track 0.00 -> 22.9 mm, vias 0 -> 2
- net /TXD: track 0.00 -> 20.3 mm
- net Net-(U3-RESET): track 0.00 -> 20.3 mm, vias 0 -> 2
- net /RXD: track 0.00 -> 15.2 mm
- net +24V: track 309.9 -> 325.1 mm
- net /SPI_SCK: track 0.00 -> 12.7 mm, vias 0 -> 2
- net /EN: track 0.00 -> 12.7 mm, vias 0 -> 5
- net /nRST: track 0.00 -> 10.2 mm, vias 0 -> 2
- net /Driver_Z/VREF: track 10.2 -> 0.00 mm
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