File: ecad/BreadBoard-POC/BreadBoard-PoC.kicad_sch (KiCad schematic)
At the start: 4 parts

Commit message: Finalizing POC placement and routing.
Parts:
- added C49, C50, C52, C54, C55, C56, C57, C58, C59: 100n, Capacitor_THT:C_Rect_L4.6mm_W2.0mm_P2.50mm_MKS02_FKP02, symbol Device:C
- added C53: 100u, Capacitor_THT:CP_Radial_D6.3mm_P2.50mm, symbol Device:C_Polarized
- added J17: AVR-ISP-6, Connector_PinHeader_2.54mm:PinHeader_2x03_P2.54mm_Vertical, symbol Connector:AVR-ISP-6
- added J18, J19, J20: Conn_01x04, Connector_PinHeader_2.54mm:PinHeader_1x04_P2.54mm_Vertical, symbol Connector_Generic:Conn_01x04
- added J21, J22: Conn_01x01, Connector_PinHeader_2.54mm:PinHeader_1x01_P2.54mm_Vertical, symbol Connector_Generic:Conn_01x01
- added R25, R36, R37, R38, R42, R43, R44: 4K7, Resistor_THT:R_Axial_DIN0207_L6.3mm_D2.5mm_P2.54mm_Vertical, symbol Device:R
- added R30, R31: 33R, Resistor_THT:R_Axial_DIN0207_L6.3mm_D2.5mm_P2.54mm_Vertical, symbol Device:R
- added R32: 10k, Resistor_THT:R_Axial_DIN0207_L6.3mm_D2.5mm_P2.54mm_Vertical, symbol Device:R
- added RN1: R_Network08, Resistor_THT:R_Array_SIP9, symbol Device:R_Network08
- added RV1: 1K, Potentiometer_THT:Potentiometer_Bourns_3266W_Vertical, symbol Device:R_Potentiometer_Trim
- added U5: ATmega328-P, Package_DIP:DIP-28_W7.62mm_LongPads, symbol MCU_Microchip_ATmega:ATmega328-P
Connections:
- net Driver_X1/VREF: now also RV1.2
- new net: J20.2 (Pin_2), R42.1, RN1.7 (R6)
- new net: J20.3 (Pin_3), R43.1, RN1.8 (R7)
- new net: J20.4 (Pin_4), R44.1, RN1.9 (R8)
- new net: J19.2 (Pin_2), R38.1, RN1.2 (R1)
- new net: J19.4 (Pin_4), R36.1, RN1.4 (R3)
- new net: J19.3 (Pin_3), R37.1, RN1.3 (R2)
- new net: R25.2, RV1.1
- new net +24V: J21.1 (Pin_1)
- new net +5V: C49.1, C50.1, C53.1, J17.2 (VCC), J18.1 (Pin_1), R25.1, R32.1, RN1.1 (common), U5.20 (AVCC), U5.7 (VCC)
- new net CYCLE_START: C54.1, R36.2, U5.25 (PC2)
- new net DIR_X: U5.11 (PD5)
- new net DIR_Y: U5.12 (PD6)
- new net DIR_Z: U5.13 (PD7)
- new net EN: U5.14 (PB0)
- new net FEED_HOLD: C55.1, R37.2, U5.24 (PC1)
- new net GND: C49.2, C50.2, C52.2, C53.2, C54.2, C55.2, C56.2, C57.2, C58.2, C59.2, J17.6 (GND), J18.4 (Pin_4), J19.1 (Pin_1), J20.1 (Pin_1), J22.1 (Pin_1), RV1.3, U5.22 (GND), U5.8 (GND)
- new net LIMIT_X: C59.1, R42.2, U5.15 (PB1)
- new net LIMIT_Y: C58.1, R43.2, U5.16 (PB2)
- new net LIMIT_Z: C57.1, R30.2, R44.2, U5.18 (PB4)
- new net RESET: C56.1, R38.2, U5.23 (PC0)
- new net RXD: J18.2 (Pin_2), U5.2 (PD0)
- new net SPINDLE_ON: R31.2, U5.17 (PB3)
- new net SPI_MISO: J17.1 (MISO), R30.1
- new net SPI_MOSI: J17.4 (MOSI), R31.1
- new net SPI_SCK: J17.3 (SCK), U5.19 (PB5)
- new net STEP_X: U5.4 (PD2)
- new net STEP_Y: U5.5 (PD3)
- new net STEP_Z: U5.6 (PD4)
- new net TXD: J18.3 (Pin_3), U5.3 (PD1)
- new net nRST: C52.1, J17.5 (~{RST}), R32.2, U5.1 (~{RESET}/PC6)
Other:
- sheet Driver_X1 ports: added none; removed RESET
- sheet Driver_X2 ports: added none; removed RESET
- sheet Driver_Y ports: added none; removed RESET
- sheet Driver_Z ports: added none; removed RESET
